File: badge/badge.kicad_sch (KiCad schematic)
At the start: 0 parts

Commit message: badge: placement mostly complete
Parts:
- added D1, D10, D11, D12, D13, D14, D15, D16, D17, D18, D19, D2, D20, D21, D22, D23, D24, D25, D26, D27, D28, D29, D3, D30, D31, D32, D33, D34, D35, D36, D4, D5, D6, D7, D8, D9: WS2812B, library:LED_WS2812B_PLCC4_5.0x5.0mm_P3.2mm, symbol library:WS2812B
Connections:
- new net: D11.2 (DOUT), D12.4 (DIN)
- new net: D10.2 (DOUT), D11.4 (DIN)
- new net: D13.2 (DOUT), D14.4 (DIN)
- new net: D12.2 (DOUT), D13.4 (DIN)
- new net: D34.2 (DOUT), D35.4 (DIN)
- new net: D33.2 (DOUT), D34.4 (DIN)
- new net: D35.2 (DOUT), D36.4 (DIN)
- new net: D1.2 (DOUT), D2.4 (DIN)
- new net: D27.2 (DOUT), D28.4 (DIN)
- new net: D26.2 (DOUT), D27.4 (DIN)
- new net: D32.2 (DOUT), D33.4 (DIN)
- new net: D4.2 (DOUT), D5.4 (DIN)
- new net: D3.2 (DOUT), D4.4 (DIN)
- new net: D25.2 (DOUT), D26.4 (DIN)
- new net: D24.2 (DOUT), D25.4 (DIN)
- new net: D23.2 (DOUT), D24.4 (DIN)
- new net: D22.2 (DOUT), D23.4 (DIN)
- new net: D31.2 (DOUT), D32.4 (DIN)
- new net: D30.2 (DOUT), D31.4 (DIN)
- new net: D14.2 (DOUT), D15.4 (DIN)
- new net: D10.4 (DIN), D9.2 (DOUT)
- new net: D8.2 (DOUT), D9.4 (DIN)
- new net: D17.2 (DOUT), D18.4 (DIN)
- new net: D16.2 (DOUT), D17.4 (DIN)
- new net: D2.2 (DOUT), D3.4 (DIN)
- new net: D5.2 (DOUT), D6.4 (DIN)
- new net: D20.2 (DOUT), D21.4 (DIN)
- new net: D19.2 (DOUT), D20.4 (DIN)
- new net: D7.2 (DOUT), D8.4 (DIN)
- new net: D29.2 (DOUT), D30.4 (DIN)
- new net: D28.2 (DOUT), D29.4 (DIN)
- new net: D15.2 (DOUT), D16.4 (DIN)
- new net: D21.2 (DOUT), D22.4 (DIN)
- new net: D6.2 (DOUT), D7.4 (DIN)
- new net: D18.2 (DOUT), D19.4 (DIN)
- new net +5V: D1.1 (VDD), D10.1 (VDD), D11.1 (VDD), D12.1 (VDD), D13.1 (VDD), D14.1 (VDD), D15.1 (VDD), D16.1 (VDD), D17.1 (VDD), D18.1 (VDD), D19.1 (VDD), D2.1 (VDD), D20.1 (VDD), D21.1 (VDD), D22.1 (VDD), D23.1 (VDD), D24.1 (VDD), D25.1 (VDD), D26.1 (VDD), D27.1 (VDD), D28.1 (VDD), D29.1 (VDD), D3.1 (VDD), D30.1 (VDD), D31.1 (VDD), D32.1 (VDD), D33.1 (VDD), D34.1 (VDD), D35.1 (VDD), D36.1 (VDD), D4.1 (VDD), D5.1 (VDD), D6.1 (VDD), D7.1 (VDD), D8.1 (VDD), D9.1 (VDD)
- new net GND: D1.3 (VSS), D10.3 (VSS), D11.3 (VSS), D12.3 (VSS), D13.3 (VSS), D14.3 (VSS), D15.3 (VSS), D16.3 (VSS), D17.3 (VSS), D18.3 (VSS), D19.3 (VSS), D2.3 (VSS), D20.3 (VSS), D21.3 (VSS), D22.3 (VSS), D23.3 (VSS), D24.3 (VSS), D25.3 (VSS), D26.3 (VSS), D27.3 (VSS), D28.3 (VSS), D29.3 (VSS), D3.3 (VSS), D30.3 (VSS), D31.3 (VSS), D32.3 (VSS), D33.3 (VSS), D34.3 (VSS), D35.3 (VSS), D36.3 (VSS), D4.3 (VSS), D5.3 (VSS), D6.3 (VSS), D7.3 (VSS), D8.3 (VSS), D9.3 (VSS)
- no-connect marks 0 -> 1

Commit message: badge: add caps for leds
Parts:
- added C1, C10, C11, C12, C13, C14, C15, C16, C17, C18, C19, C2, C20, C21, C22, C23, C24, C25, C26, C27, C28, C29, C3, C30, C31, C32, C33, C34, C35, C36, C4, C5, C6, C7, C8, C9: 100nF,16V,X7R, C_0402_1005Metric, symbol library:100nF,16V,X7R
Connections:
- net +5V: now also C1.1, C10.1, C11.1, C12.1, C13.1, C14.1, C15.1, C16.1, C17.1, C18.1, C19.1, C2.1, C20.1, C21.1, C22.1, C23.1, C24.1, C25.1, C26.1, C27.1, C28.1, C29.1, C3.1, C30.1, C31.1, C32.1, C33.1, C34.1, C35.1, C36.1, C4.1, C5.1, C6.1, C7.1, C8.1, C9.1
- net GND: now also C17.2, C18.2, C19.2, C20.2, C21.2, C22.2, C23.2, C24.2, C25.2, C26.2, C27.2, C28.2, C29.2, C30.2, C31.2, C32.2, C35.2, C36.2
- new net: C1.2, C10.2, C11.2, C12.2, C13.2, C14.2, C15.2, C16.2, C2.2, C3.2, C33.2, C34.2, C4.2, C5.2, C6.2, C7.2, C8.2, C9.2
Other:
- moved on the sheet: D1, D10, D11, D12, D13, D14, D15, D16, D17, D18, D19, D2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

Commit message: badeg: complete
Parts:
- added C37: 100nF,16V,X7R, library:C_0402_1005Metric, symbol library:100nF,16V,X7R
- added C38: 10uF,10V,X5R, library:C_0603_1608Metric, symbol library:10uF,10V,X5R
- added J1: Conn_01x03, library:PinHeader_1x03_P2.54mm_Horizontal_SMD, symbol library:Conn_01x03
- added U1: 74LVC1G125, library:SOT-23-5, symbol library:74LVC1G125
- C1, C10, C11, C12, C13, C14, C15, C16, C17, C18, C19, C2, C20, C21, C22, C23, C24, C25, C26, C27, C28, C29, C3, C30, C31, C32, C33, C34, C35, C36, C4, C5, C6, C7, C8, C9: footprint C_0402_1005Metric -> library:C_0402_1005Metric
Connections:
- net +5V: now also C37.1, C38.1, J1.1 (Pin_1), U1.5 (VCC)
- net GND: now also C1.2, C10.2, C11.2, C12.2, C13.2, C14.2, C15.2, C16.2, C2.2, C3.2, C33.2, C34.2, C4.2, C5.2, C6.2, C7.2, C8.2, C9.2, C37.2, C38.2, J1.2 (Pin_2), U1.1, U1.3 (GND)
- net at D1.4 (DIN): now also U1.4
- new net: J1.3 (Pin_3), U1.2
Other:
- moved on the sheet: C1, C10, C11, C12, C13, C14, C15, C16, C17, C18, C19, C2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

Commit message: badge: ver 1.1 ready for production
Parts:
- added J2: Conn_01x03, library:PinHeader_1x03_P2.54mm_Horizontal_SMD, symbol library:Conn_01x03
- J1: now left out of the parts list
Connections:
- net +5V: now also J2.3 (Pin_3)
- net GND: now also J2.2 (Pin_2)
- net at J1.3 (Pin_3), U1.2: now also J2.1 (Pin_1)
Changed lines of the file:
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@@
   (junction (at 127.635 35.56) (diameter 0) (color 0 0 0 0)
+  )
+  (junction (at 47.625 85.725) (diameter 0) (color 0 0 0 0)
   )
   (junction (at 159.385 76.835) (diameter 0) (color 0 0 0 0)
@@
     (stroke (width 0) (type default))
   )
+  (wire (pts (xy 47.625 111.125) (xy 47.625 85.725))
+    (stroke (width 0) (type default))
+  )
   (wire (pts (xy 113.665 106.045) (xy 113.665 107.315))
     (stroke (width 0) (type default))
@@
     (stroke (width 0) (type default))
   )
+  (wire (pts (xy 36.195 116.205) (xy 38.1 116.205))
+    (stroke (width 0) (type default))
+  )
   (wire (pts (xy 82.55 167.64) (xy 82.55 168.91))
     (stroke (width 0) (type default))
@@
     (stroke (width 0) (type default))
   )
+  (wire (pts (xy 36.195 111.125) (xy 47.625 111.125))
+    (stroke (width 0) (type default))
+  )
   (wire (pts (xy 198.755 64.135) (xy 189.865 64.135))
     (stroke (width 0) (type default))
@@
   )
   (wire (pts (xy 173.99 153.67) (xy 173.99 154.94))
+    (stroke (width 0) (type default))
+  )
+  (wire (pts (xy 36.195 113.665) (xy 38.1 113.665))
     (stroke (width 0) (type default))
   )
@@
   )
   (symbol (lib_id "library:Conn_01x03") (at 31.115 83.185 0) (mirror y) (unit 1)
-    (in_bom yes) (on_board yes) (dnp no) (fields_autoplaced)
+    (in_bom no) (on_board yes) (dnp no) (fields_autoplaced)
     (property "Reference" "J1" (at 31.115 75.565 0)
       (effects (font (size 1.27 1.27)))
@@
     )
   )
+  (symbol (lib_id "library:Conn_01x03") (at 31.115 113.665 0) (mirror y) (unit 1)
+    (in_bom no) (on_board yes) (dnp no) (fields_autoplaced)
+    (property "Reference" "J2" (at 31.115 106.045 0)
+      (effects (font (size 1.27 1.27)))
+    )
+    (property "Value" "Conn_01x03" (at 31.115 108.585 0)
+      (effects (font (size 1.27 1.27)))
+    )
+    (property "Footprint" "library:PinHeader_1x03_P2.54mm_Horizontal_SMD" (at 31.115 113.665 0)
+      (effects (font (size 1.27 1.27)) hide)
+    )
+    (property "Datasheet" "~" (at 31.115 113.665 0)
+      (effects (font (size 1.27 1.27)) hide)
+    )
+    (pin "1")
+    (pin "2")
+    (pin "3")
+    (instances
+      (project "badge"
+        (path "/7d02ad2e-1319-4c8b-85de-c3995a559434"
+          (reference "J2") (unit 1)
+        )
+      )
+    )
+  )
   (symbol (lib_id "library:WS2812B") (at 205.105 85.725 0) (unit 1)
     (in_bom yes) (on_board yes) (dnp no)
@@
     )
   )
+  (symbol (lib_id "power:GND") (at 38.1 113.665 90) (unit 1)
+    (in_bom yes) (on_board yes) (dnp no)
+    (property "Reference" "#PWR022" (at 44.45 113.665 0)
+      (effects (font (size 1.27 1.27)) hide)
+    )
+    (property "Value" "GND" (at 43.18 113.665 90)
+      (effects (font (size 1.27 1.27)))
+    )
+    (property "Footprint" "" (at 38.1 113.665 0)
+      (effects (font (size 1.27 1.27)) hide)
+    )
+    (property "Datasheet" "" (at 38.1 113.665 0)
+      (effects (font (size 1.27 1.27)) hide)
+    )
+    (pin "1")
+    (instances
+      (project "badge"
+        (path "/7d02ad2e-1319-4c8b-85de-c3995a559434"
+          (reference "#PWR022") (unit 1)
+        )
+      )
+    )
+  )
   (symbol (lib_id "power:+5V") (at 83.185 106.045 0) (unit 1)
     (in_bom yes) (on_board yes) (dnp no) (fields_autoplaced)
@@
         )
       )
+    )
+  )
+  (symbol (lib_id "power:+5V") (at 38.1 116.205 270) (unit 1)
+    (in_bom yes) (on_board yes) (dnp no) (fields_autoplaced)
+    (property "Reference" "#PWR021" (at 34.29 116.205 0)
+      (effects (font (size 1.27 1.27)) hide)
+    )
+    (property "Value" "+5V" (at 41.275 116.84 90)
+      (effects (font (size 1.27 1.27)) (justify left))
+    )
+    (property "Footprint" "" (at 38.1 116.205 0)
+      (effects (font (size 1.27 1.27)) hide)
+    )
+    (property "Datasheet" "" (at 38.1 116.205 0)
+      (effects (font (size 1.27 1.27)) hide)
+    )
+    (pin "1")
+    (instances
+      (project "badge"
+        (path "/7d02ad2e-1319-4c8b-85de-c3995a559434"
+          (reference "#PWR021") (unit 1)
+        )
+      )
